Commit message: add color

File: URDF/gankenkun.urdf (robot description, URDF)
Before this commit: robot gankenkun, 35 links, 34 joints
Links:
- link body_link: geometry collision mesh filename=URDF/meshes/STL/body.stl; visual mesh filename=URDF/meshes/STL/body.stl
- link head_yaw_link: geometry collision mesh filename=URDF/meshes/STL/head.stl; visual mesh filename=URDF/meshes/STL/head.stl
- link left_ankle_pitch_link: geometry collision mesh filename=URDF/meshes/STL/ankle_pitch_left.stl; visual mesh filename=URDF/meshes/STL/ankle_pitch_left.stl
- link left_ankle_roll_link: geometry collision mesh filename=URDF/meshes/STL/ankle_roll_left.stl; visual mesh filename=URDF/meshes/STL/ankle_roll_left.stl
- link left_independent_pitch_link: geometry collision mesh filename=URDF/meshes/STL/independent_pitch.stl; visual mesh filename=URDF/meshes/STL/independent_pitch.stl
- link left_knee_pitch_link: geometry collision mesh filename=URDF/meshes/STL/knee_pitch_left.stl; visual mesh filename=URDF/meshes/STL/knee_pitch_left.stl
- link left_lower_arm_link: geometry collision mesh filename=URDF/meshes/STL/hand.stl; visual mesh filename=URDF/meshes/STL/hand.stl
- link left_shin_pitch_link: geometry collision mesh filename=URDF/meshes/STL/shin_pitch.stl; visual mesh filename=URDF/meshes/STL/shin_pitch.stl
- link left_shin_pitch_mimic_link: geometry collision mesh filename=URDF/meshes/STL/shin_pitch_mimic.stl; visual mesh filename=URDF/meshes/STL/shin_pitch_mimic.stl
- link left_shoulder_link: geometry collision mesh filename=URDF/meshes/STL/shoulder.stl; visual mesh filename=URDF/meshes/STL/shoulder.stl
- link left_slider_crank_link: geometry collision mesh filename=URDF/meshes/STL/slider_crank.stl; visual mesh filename=URDF/meshes/STL/slider_crank.stl
- link left_upper_arm_link: geometry collision mesh filename=URDF/meshes/STL/arm.stl; visual mesh filename=URDF/meshes/STL/arm.stl
- link left_waist_pitch_link: geometry collision mesh filename=URDF/meshes/STL/waist_pitch.stl; visual mesh filename=URDF/meshes/STL/waist_pitch.stl
- link left_waist_pitch_mimic_link: geometry collision mesh filename=URDF/meshes/STL/waist_pitch_mimic.stl; visual mesh filename=URDF/meshes/STL/waist_pitch_mimic.stl
- link left_waist_roll_link: geometry collision mesh filename=URDF/meshes/STL/waist_roll_left.stl; visual mesh filename=URDF/meshes/STL/waist_roll_left.stl
- link left_waist_yaw_link: geometry collision mesh filename=URDF/meshes/STL/waist_yaw.stl; visual mesh filename=URDF/meshes/STL/waist_yaw.stl
- link right_ankle_pitch_link: geometry collision mesh filename=URDF/meshes/STL/ankle_pitch_right.stl; visual mesh filename=URDF/meshes/STL/ankle_pitch_right.stl
- link right_ankle_roll_link: geometry collision mesh filename=URDF/meshes/STL/ankle_roll_right.stl; visual mesh filename=URDF/meshes/STL/ankle_roll_right.stl
- link right_independent_pitch_link: geometry collision mesh filename=URDF/meshes/STL/independent_pitch.stl; visual mesh filename=URDF/meshes/STL/independent_pitch.stl
- link right_knee_pitch_link: geometry collision mesh filename=URDF/meshes/STL/knee_pitch_right.stl; visual mesh filename=URDF/meshes/STL/knee_pitch_right.stl
- link right_lower_arm_link: geometry collision mesh filename=URDF/meshes/STL/hand.stl; visual mesh filename=URDF/meshes/STL/hand.stl
- link right_shin_pitch_link: geometry collision mesh filename=URDF/meshes/STL/shin_pitch.stl; visual mesh filename=URDF/meshes/STL/shin_pitch.stl
- link right_shin_pitch_mimic_link: geometry collision mesh filename=URDF/meshes/STL/shin_pitch_mimic.stl; visual mesh filename=URDF/meshes/STL/shin_pitch_mimic.stl
- link right_shoulder_link: geometry collision mesh filename=URDF/meshes/STL/shoulder.stl; visual mesh filename=URDF/meshes/STL/shoulder.stl
- link right_slider_crank_link: geometry collision mesh filename=URDF/meshes/STL/slider_crank.stl; visual mesh filename=URDF/meshes/STL/slider_crank.stl
- link right_upper_arm_link: geometry collision mesh filename=URDF/meshes/STL/arm.stl; visual mesh filename=URDF/meshes/STL/arm.stl
- link right_waist_pitch_link: geometry collision mesh filename=URDF/meshes/STL/waist_pitch.stl; visual mesh filename=URDF/meshes/STL/waist_pitch.stl
- link right_waist_pitch_mimic_link: geometry collision mesh filename=URDF/meshes/STL/waist_pitch_mimic.stl; visual mesh filename=URDF/meshes/STL/waist_pitch_mimic.stl
- link right_waist_roll_link: geometry collision mesh filename=URDF/meshes/STL/waist_roll_right.stl; visual mesh filename=URDF/meshes/STL/waist_roll_right.stl
- link right_waist_yaw_link: geometry collision mesh filename=URDF/meshes/STL/waist_yaw.stl; visual mesh filename=URDF/meshes/STL/waist_yaw.stl

File: URDF/plane.urdf (robot description, URDF)
Before this commit: robot plane, 1 links, 0 joints
Links:
- link planeLink: geometry collision box size=30 30 10; visual mesh filename=plane.obj scale=1 1 1

Commit message: get correct image

File: URDF/gankenkun.urdf (robot description, URDF)
Before this commit: robot gankenkun, 35 links, 34 joints
Joints:
- joint camera_joint: origin xyz=0.036495 0 0.063504 rpy=0 0.785398163397 0 -> xyz=0.036495 0 0.063504 rpy=0.785398163397 0 -1.5707963268

Commit message: change inertia

File: URDF/gankenkun.urdf (robot description, URDF)
Before this commit: robot gankenkun, 35 links, 34 joints
Links:
- link camera_link: mass None -> 0.0
- link imu_link: mass None -> 0.0
- link left_foot_link: mass None -> 0.0
- link right_foot_link: mass None -> 0.0
